Commit message: gps waypoint configured
Minor error still there

File: bot_description/urdf/bot.urdf.xacro (robot description, xacro)
@@ -264,4 +264,21 @@
   <link name="navsat_link">
   </link>
+  <joint name="imu_joint" type="fixed">
+    <origin xyz="0 0 0" rpy="0 0 0" />
+    <parent link="base_link"/>
+    <child link="imu_link" />
+  </joint>
+  <link name="imu_link">
+  </link>
+  <gazebo reference="imu_link">
+    <sensor name="imu" type="imu">
+      <always_on>1</always_on>
+      <update_rate>50</update_rate>
+      <visualize>true</visualize>
+      <topic>imu</topic>
+      <enable_metrics>true</enable_metrics>
+      <gz_frame_id>imu_link</gz_frame_id>
+    </sensor>
+  </gazebo>
   <gazebo reference="navsat_link">
     <sensor name="navsat" type="navsat">

Commit message: start qr code replacement
key issue - moderate drift in odometry and jitters in autonomous nav

File: bot_description/urdf/bot.urdf.xacro (robot description, xacro)
@@ -3,9 +3,4 @@
   <xacro:include filename="bot_ros2_control.xacro" />
   <link name="base_footprint">
-      <inertial>
-            <mass value="2" />
-            <inertia ixx="0.04" ixy="0.0" ixz="0"
-            iyy="0.17" iyz="0" izz="0.25" />
-    </inertial>
   </link>
   <joint name="base_joint" type="fixed">
@@ -14,107 +9,115 @@
     <origin xyz="0.0 0.0 0.15" rpy="0.0 0.0 3.14159"/>
   </joint>
-  <link name="base_link">
-    <visual>
-      <geometry>
-          <box size=".8 0.7 0.2"/>
-      </geometry>
-      <material name="gray">
-        <color rgba=".2 .2 .2 1" />
-      </material>
-    </visual>
-    <inertial>
-            <mass value="2" />
-            <inertia ixx="0.04" ixy="0.0" ixz="0"
-            iyy="0.17" iyz="0" izz="0.25" />
-    </inertial>
-    <collision>
-      <geometry>
-          <box size=".8 0.7 0.2"/>
-      </geometry>
-    </collision>
-  </link>
+<link name="base_link">
+  <visual>
+    <geometry>
+      <box size="0.8 0.7 0.2"/>
+    </geometry>
+    <material name="gray">
+      <color rgba="0.2 0.2 0.2 1" />
+    </material>
+  </visual>
+  <collision>
+    <geometry>
+      <box size="0.8 0.7 0.2"/>
+    </geometry>
+  </collision>
+  <inertial>
+    <mass value="2"/>
+    <inertia ixx="0.0883" ixy="0.0" ixz="0.0"
+             iyy="0.1133" iyz="0.0" izz="0.187"/>
+  </inertial>
+</link>
   <link name="wheel_front_right">
-    <inertial>
-            <mass value="2" />
-            <inertia ixx="1e-3" ixy="0.0" ixz="0"
-            iyy="1e-3" iyz="0" izz="1e-3" />
-    </inertial>
-    <visual>
-      <geometry>
-          <cylinder radius="0.10" length="0.1"/>
-      </geometry>
-      <material name="white">
-        <color rgba="1 1 1 1"/>
-      </material>
-    </visual>
-    <collision>
-      <geometry>
-          <sphere radius="0.10"/>
-      </geometry>
-    </collision>
+  <inertial>
+    <mass value="0.5"/>  <!-- OK for small wheels -->
+    <inertia
+      ixx="0.00025" ixy="0.0" ixz="0.0"
+      iyy="0.00025" iyz="0.0"
+      izz="0.0001"/>
+  </inertial>
+  <visual>
+    <geometry>
+      <cylinder radius="0.10" length="0.05"/>
+    </geometry>
+    <material name="white">
+      <color rgba="1 1 1 1"/>
+    </material>
+  </visual>
+  <collision>
+    <geometry>
+      <cylinder radius="0.10" length="0.05"/>
+    </geometry>
+  </collision>
   </link>
   <link name="wheel_front_left">
-    <inertial>
-            <mass value="2" />
-            <inertia ixx="1e-3" ixy="0.0" ixz="0"
-            iyy="1e-3" iyz="0" izz="1e-3" />
-    </inertial>
-    <visual>
-      <geometry>
-          <cylinder radius="0.10" length="0.1"/>
-      </geometry>
-      <material name="white">
-        <color rgba="1 1 1 1"/>
-      </material>
-    </visual>
-    <collision>
-      <geometry>
-          <sphere radius="0.10" />
-      </geometry>
-    </collision>
+  <inertial>
+    <mass value="0.5"/>  <!-- OK for small wheels -->
+    <inertia
+      ixx="0.00025" ixy="0.0" ixz="0.0"
+      iyy="0.00025" iyz="0.0"
+      izz="0.0001"/>
+  </inertial>
+  <visual>
+    <geometry>
+      <cylinder radius="0.10" length="0.05"/>
+    </geometry>
+    <material name="white">
+      <color rgba="1 1 1 1"/>
+    </material>
+  </visual>
+  <collision>
+    <geometry>
+      <cylinder radius="0.10" length="0.05"/>
+    </geometry>
+  </collision>
   </link>
 <link name="wheel_back_right">
-    <inertial>
-            <mass value="2" />
-            <inertia ixx="1e-3" ixy="0.0" ixz="0"
-            iyy="1e-3" iyz="0" izz="1e-3" />
-    </inertial>
-    <visual>
-      <geometry>
-          <cylinder radius="0.10" length="0.1"/>
-      </geometry>
-      <material name="white">
-        <color rgba="1 1 1 1"/>
-      </material>
-    </visual>
-    <collision>
-      <geometry>
-          <sphere radius="0.10" />
-      </geometry>
-    </collision>
-  </link>
-  <link name="wheel_back_left">
-    <inertial>
-            <mass value="2" />
-            <inertia ixx="1e-3" ixy="0.0" ixz="0"
-            iyy="1e-3" iyz="0" izz="1e-3" />
-    </inertial>
-    <visual>
-      <geometry>
-          <cylinder radius="0.10" length="0.1"/>
-      </geometry>
-      <material name="white">
-        <color rgba="1 1 1 1"/>
-      </material>
-    </visual>
-    <collision>
-      <geometry>
-          <sphere radius="0.10"/>
-      </geometry>
-    </collision>
-  </link>
+  <inertial>
+    <mass value="0.5"/>  <!-- OK for small wheels -->
+    <inertia
+      ixx="0.00025" ixy="0.0" ixz="0.0"
+      iyy="0.00025" iyz="0.0"
+      izz="0.0001"/>
+  </inertial>
+  <visual>
+    <geometry>
+      <cylinder radius="0.10" length="0.05"/>
+    </geometry>
+    <material name="white">
+      <color rgba="1 1 1 1"/>
+    </material>
+  </visual>
+  <collision>
+    <geometry>
+      <cylinder radius="0.10" length="0.05"/>
+    </geometry>
+  </collision>
+  </link>
+<link name="wheel_back_left">
+  <inertial>
+    <mass value="0.5"/>
+    <inertia
+      ixx="0.00025" ixy="0.0" ixz="0.0"
+      iyy="0.00025" iyz="0.0"
+      izz="0.0001"/>
+  </inertial>
+  <visual>
+    <geometry>
+      <cylinder radius="0.10" length="0.05"/>
+    </geometry>
+    <material name="white">
+      <color rgba="1 1 1 1"/>
+    </material>
+  </visual>
+  <collision>
+    <geometry>
+      <cylinder radius="0.10" length="0.05"/>
+    </geometry>
+  </collision>
+</link>
   <link name="rgb_camera">
     <inertial>
-            <mass value="0.5" />
+            <mass value="0.05" />
             <inertia ixx="0.01" ixy="0.0" ixz="0"
             iyy="0.01" iyz="0" izz="0.01" />
@@ -140,28 +143,37 @@
     <axis xyz="0.0 0 0"/>
   </joint>
+  <joint type="fixed" name="camera_optical_joint">
+    <origin xyz="0 0 0" rpy="-1.5707 0 -1.5707"/>
+    <child link="camera_link_optical"/>
+    <parent link="rgb_camera"/>
+  </joint>
+  <link name="camera_link_optical">
+  </link>
     <gazebo reference="rgb_camera">
-        <sensor name="camera" type="camera">
-            <always_on>true</always_on>
-            <update_rate>30.0</update_rate>
-            <visualize>true</visualize>
-            <topic>/camera/image_raw</topic>
-            <gz_frame_id>/rgb_camera</gz_frame_id>
-            <camera name="camera">
-            <horizontal_fov>1.21126</horizontal_fov>
-            <image>
-                <width>640</width>
-                <height>640</height>
-                <format>R8G8B8</format>
-            </image>
-            <distortion>
-                <k1>0.0</k1>
-                <k2>0.0</k2>
-                <k3>0.0</k3>
-                <p1>0.0</p1>
-                <p2>0.0</p2>
-                <center>0.5 0.5</center>
-            </distortion>
-            </camera>
-        </sensor>
+    <sensor name="camera" type="camera">
+      <camera>
+        <horizontal_fov>1.3962634</horizontal_fov>
+        <image>
+          <width>640</width>
+          <height>480</height>
+          <format>R8G8B8</format>
+        </image>
+        <clip>
+          <near>0.1</near>
+          <far>15</far>
+        </clip>
+        <noise>
+          <type>gaussian</type>
+          <mean>0.0</mean>
+          <stddev>0.007</stddev>
+        </noise>
+        <optical_frame_id>camera_link_optical</optical_frame_id>
+        <camera_info_topic>camera/camera_info</camera_info_topic>
+      </camera>
+      <always_on>1</always_on>
+      <update_rate>20</update_rate>
+      <visualize>true</visualize>
+      <topic>camera/image_raw</topic>
+    </sensor>
     </gazebo>
   <link name="laser_link">
@@ -192,5 +204,5 @@
   </joint>
     <!-- 2D LIDAR-->
-<!--  <gazebo reference="laser_link">
+  <gazebo reference="laser_link">
     <sensor name="lidar" type="gpu_lidar">
       <always_on>true</always_on>
@@ -220,40 +232,4 @@
       </lidar>
     </sensor>
-  </gazebo>-->
-  <!-- velodyne vlp-32 3D lidar plugin-->
-  <gazebo reference="laser_link">
-    <sensor name="lidar" type="gpu_lidar">
-      <update_rate>10</update_rate>
-      <topic>scan</topic>
-      <gz_frame_id>laser_link</gz_frame_id>
-      <lidar>
-        <scan>
-          <horizontal>
-            <samples>720</samples>
-            <resolution>1</resolution>
-            <min_angle>-3.14156</min_angle>
-            <max_angle>3.14156</max_angle>
-          </horizontal>
-          <vertical>
-            <samples>32</samples>
-            <min_angle>-0.5353</min_angle>
-            <max_angle>0.1862</max_angle>
-          </vertical>
-        </scan>
-        <range>
-          <min>0.05</min>
-          <max>10.0</max>
-          <resolution>0.01</resolution>
-        </range>
-        <noise>
-            <type>gaussian</type>
-            <mean>0.0</mean>
-            <stddev>0.01</stddev>
-        </noise>
-        <frame_id>scan_link</frame_id>
-      </lidar>
-      <always_on>1</always_on>
-      <visualize>true</visualize>
-    </sensor>
   </gazebo>
   <joint name="navsat_joint" type="fixed">
@@ -314,37 +290,37 @@
   </joint>
     <gazebo reference="wheel_front_right">
-    <mu1>1000000000000000.0</mu1>
-    <mu2>1000000000000000.0</mu2>
-    <kp>1000000000000.0</kp>
-    <kd>10.0</kd>
+    <mu1>1.0</mu1>
+    <mu2>0.8</mu2>
+    <kp>100000.0</kp>
+    <kd>1.0</kd>
     <minDepth>0.001</minDepth>
-    <maxVel>0.1</maxVel>
+    <maxVel>1</maxVel>
     <fdir1>1 0 0</fdir1>
     </gazebo>
     <gazebo reference="wheel_front_left">
-    <mu1>1000000000000000.0</mu1>
-    <mu2>1000000000000000.0</mu2>
-    <kp>1000000000000.0</kp>
-    <kd>10.0</kd>
+    <mu1>1.0</mu1>
+    <mu2>0.8</mu2>
+    <kp>100000.0</kp>
+    <kd>1.0</kd>
     <minDepth>0.001</minDepth>
-    <maxVel>0.1</maxVel>
+    <maxVel>1</maxVel>
     <fdir1>1 0 0</fdir1>
     </gazebo>
     <gazebo reference="wheel_back_right">
-    <mu1>1000000000000000.0</mu1>
-    <mu2>1000000000000000.0</mu2>
-    <kp>1000000000000.0</kp>
-    <kd>10.0</kd>
+    <mu1>1.0</mu1>
+    <mu2>0.8</mu2>
+    <kp>100000.0</kp>
+    <kd>1.0</kd>
     <minDepth>0.001</minDepth>
-    <maxVel>0.1</maxVel>
+    <maxVel>1</maxVel>
     <fdir1>1 0 0</fdir1>
     </gazebo>
     <gazebo reference="wheel_back_left">
-    <mu1>1000000000000000.0</mu1>
-    <mu2>1000000000000000.0</mu2>
-    <kp>1000000000000.0</kp>
-    <kd>10.0</kd>
+    <mu1>1.0</mu1>
+    <mu2>0.8</mu2>
+    <kp>100000.0</kp>
+    <kd>1.0</kd>
     <minDepth>0.001</minDepth>
-    <maxVel>0.1</maxVel>
+    <maxVel>1</maxVel>
     <fdir1>1 0 0</fdir1>
     </gazebo>

Commit message: new baylands world integrated

File: bot_description/urdf/bot.urdf.xacro (robot description, xacro)
@@ -25,6 +25,5 @@
   <inertial>
     <mass value="2"/>
-    <inertia ixx="0.0883" ixy="0.0" ixz="0.0"
-             iyy="0.1133" iyz="0.0" izz="0.187"/>
+    <inertia ixx="0.0817" iyy="0.1067" izz="0.18" ixy="0.0" ixz="0.0" iyz="0.0"/>
   </inertial>
 </link>
@@ -32,8 +31,5 @@
   <inertial>
     <mass value="0.5"/>  <!-- OK for small wheels -->
-    <inertia
-      ixx="0.00025" ixy="0.0" ixz="0.0"
-      iyy="0.00025" iyz="0.0"
-      izz="0.0001"/>
+    <inertia ixx="0.00156" iyy="0.00156" izz="0.0025" ixy="0.0" ixz="0.0" iyz="0.0"/>
   </inertial>
   <visual>
@@ -54,8 +50,5 @@
   <inertial>
     <mass value="0.5"/>  <!-- OK for small wheels -->
-    <inertia
-      ixx="0.00025" ixy="0.0" ixz="0.0"
-      iyy="0.00025" iyz="0.0"
-      izz="0.0001"/>
+    <inertia ixx="0.00156" iyy="0.00156" izz="0.0025" ixy="0.0" ixz="0.0" iyz="0.0"/>
   </inertial>
   <visual>
@@ -76,8 +69,5 @@
   <inertial>
     <mass value="0.5"/>  <!-- OK for small wheels -->
-    <inertia
-      ixx="0.00025" ixy="0.0" ixz="0.0"
-      iyy="0.00025" iyz="0.0"
-      izz="0.0001"/>
+    <inertia ixx="0.00156" iyy="0.00156" izz="0.0025" ixy="0.0" ixz="0.0" iyz="0.0"/>
   </inertial>
   <visual>
@@ -98,8 +88,5 @@
   <inertial>
     <mass value="0.5"/>
-    <inertia
-      ixx="0.00025" ixy="0.0" ixz="0.0"
-      iyy="0.00025" iyz="0.0"
-      izz="0.0001"/>
+    <inertia ixx="0.00156" iyy="0.00156" izz="0.0025" ixy="0.0" ixz="0.0" iyz="0.0"/>
   </inertial>
   <visual>
@@ -133,5 +120,5 @@
     <collision>
       <geometry>
-          <box size="0.1 0.5 0.2"/>
+          <box size="0.1 0.1 0.1"/>
       </geometry>
     </collision>
@@ -293,5 +280,5 @@
     <mu2>0.8</mu2>
     <kp>100000.0</kp>
-    <kd>1.0</kd>
+    <kd>10.0</kd>
     <minDepth>0.001</minDepth>
     <maxVel>1</maxVel>
@@ -302,5 +289,5 @@
     <mu2>0.8</mu2>
     <kp>100000.0</kp>
-    <kd>1.0</kd>
+    <kd>10.0</kd>
     <minDepth>0.001</minDepth>
     <maxVel>1</maxVel>
@@ -311,5 +298,5 @@
     <mu2>0.8</mu2>
     <kp>100000.0</kp>
-    <kd>1.0</kd>
+    <kd>10.0</kd>
     <minDepth>0.001</minDepth>
     <maxVel>1</maxVel>
@@ -320,5 +307,5 @@
     <mu2>0.8</mu2>
     <kp>100000.0</kp>
-    <kd>1.0</kd>
+    <kd>10.0</kd>
     <minDepth>0.001</minDepth>
     <maxVel>1</maxVel>

Commit message: ekf configured

File: bot_description/urdf/bot.urdf.xacro (robot description, xacro)
@@ -49,5 +49,5 @@
   <link name="wheel_front_left">
   <inertial>
-    <mass value="0.5"/>  <!-- OK for small wheels -->
+    <mass value="0.5"/>
     <inertia ixx="0.00156" iyy="0.00156" izz="0.0025" ixy="0.0" ixz="0.0" iyz="0.0"/>
   </inertial>
@@ -68,5 +68,5 @@
 <link name="wheel_back_right">
   <inertial>
-    <mass value="0.5"/>  <!-- OK for small wheels -->
+    <mass value="0.5"/>
     <inertia ixx="0.00156" iyy="0.00156" izz="0.0025" ixy="0.0" ixz="0.0" iyz="0.0"/>
   </inertial>
@@ -191,5 +191,5 @@
   </joint>
     <!-- 2D LIDAR-->
-  <gazebo reference="laser_link">
+<!--  <gazebo reference="laser_link">
     <sensor name="lidar" type="gpu_lidar">
       <always_on>true</always_on>
@@ -219,4 +219,40 @@
       </lidar>
     </sensor>
+  </gazebo>-->
+    <!-- velodyne vlp-32 3D lidar plugin-->
+  <gazebo reference="laser_link">
+    <sensor name="lidar" type="gpu_lidar">
+      <update_rate>10</update_rate>
+      <topic>scan</topic>
+      <gz_frame_id>laser_link</gz_frame_id>
+      <lidar>
+        <scan>
+          <horizontal>
+            <samples>720</samples>
+            <resolution>1</resolution>
+            <min_angle>-3.14156</min_angle>
+            <max_angle>3.14156</max_angle>
+          </horizontal>
+          <vertical>
+            <samples>32</samples>
+            <min_angle>-0.5353</min_angle>
+            <max_angle>0.1862</max_angle>
+          </vertical>
+        </scan>
+        <range>
+          <min>0.05</min>
+          <max>50.0</max>
+          <resolution>0.01</resolution>
+        </range>
+        <noise>
+            <type>gaussian</type>
+            <mean>0.0</mean>
+            <stddev>0.01</stddev>
+        </noise>
+        <frame_id>scan_link</frame_id>
+      </lidar>
+      <always_on>1</always_on>
+      <visualize>true</visualize>
+    </sensor>
   </gazebo>
   <joint name="navsat_joint" type="fixed">
@@ -234,14 +270,54 @@
   <link name="imu_link">
   </link>
-  <gazebo reference="imu_link">
-    <sensor name="imu" type="imu">
-      <always_on>1</always_on>
-      <update_rate>50</update_rate>
-      <visualize>true</visualize>
-      <topic>imu</topic>
-      <enable_metrics>true</enable_metrics>
-      <gz_frame_id>imu_link</gz_frame_id>
-    </sensor>
-  </gazebo>
+   <gazebo reference="imu_link">
+      <sensor name="imu" type="imu">
+          <always_on>true</always_on>
+          <update_rate>100</update_rate>
+          <gz_frame_id>imu_link</gz_frame_id>
+          <topic>imu</topic>
+          <imu>
+            <angular_velocity>
+              <x>
+                <noise type="gaussian">
+                  <mean>0.0</mean>
+                  <stddev>2e-4</stddev>
+                </noise>
+              </x>
+              <y>
+                <noise type="gaussian">
+                  <mean>0.0</mean>
+                  <stddev>2e-4</stddev>
+                </noise>
+              </y>
+              <z>
+                <noise type="gaussian">
+                  <mean>0.0</mean>
+                  <stddev>2e-4</stddev>
+                </noise>
+              </z>
+            </angular_velocity>
+            <linear_acceleration>
+              <x>
+                <noise type="gaussian">
+                  <mean>0.0</mean>
+                  <stddev>1.7e-2</stddev>
+                </noise>
+              </x>
+              <y>
+                <noise type="gaussian">
+                  <mean>0.0</mean>
+                  <stddev>1.7e-2</stddev>
+                </noise>
+              </y>
+              <z>
+                <noise type="gaussian">
+                  <mean>0.0</mean>
+                  <stddev>1.7e-2</stddev>
+                </noise>
+              </z>
+            </linear_acceleration>
+          </imu>
+      </sensor>
+    </gazebo>
   <gazebo reference="navsat_link">
     <sensor name="navsat" type="navsat">

Commit message: thermal + aerial cam

File: bot_description/urdf/bot.urdf.xacro (robot description, xacro)
@@ -164,4 +164,57 @@
     </sensor>
     </gazebo>
+  <link name="thermal_camera">
+    <inertial>
+            <mass value="0.05" />
+            <inertia ixx="0.01" ixy="0.0" ixz="0"
+            iyy="0.01" iyz="0" izz="0.01" />
+    </inertial>
+    <visual>
+      <geometry>
+        <box size="0.1 0.1 0.1"/>
+      </geometry>
+      <material name="blue">
+        <color rgba="0 0 1 1"/>
+      </material>
+    </visual>    <origin xyz="-0.35 0 0.15" rpy="0 0.0 3.14"/>
+    <collision>
+      <geometry>
+          <box size="0.1 0.1 0.1"/>
+      </geometry>
+    </collision>
+  </link>
+  <joint name="thermal_camera_joint" type="fixed">
+    <origin xyz="-0.43 0 0.15" rpy="0 0.0 3.14"/>
+    <parent link="base_link"/>
+    <child link="thermal_camera"/>
+    <axis xyz="0.0 0 0"/>
+  </joint>
+  <gazebo reference="thermal_camera">
+    <sensor name="thermal_camera_8bit" type="thermal">
+      <camera>
+        <horizontal_fov>1.047</horizontal_fov>
+        <image>
+          <width>320</width>
+          <height>240</height>
+          <format>L8</format>
+        </image>
+        <clip>
+          <near>0.1</near>
+          <far>100</far>
+        </clip>
+      </camera>
+      <always_on>1</always_on>
+      <update_rate>30</update_rate>
+      <visualize>true</visualize>
+      <topic>thermal_camera_8bit/image</topic>
+      <plugin
+        filename="ignition-gazebo-thermal-sensor-system"
+        name="gz::sim::systems::ThermalSensor">
+        <min_temp>253.15</min_temp>
+        <max_temp>673.15</max_temp>
+        <resolution>3.0</resolution>
+      </plugin>
+    </sensor>
+  </gazebo>
   <link name="laser_link">
     <inertial>
@@ -185,10 +238,10 @@
   </link>
   <joint name="laser_joint" type="fixed">
-    <origin xyz="0 0 0.15" rpy="0 0.0 3.14"/>
+    <origin xyz="0 0 0.3" rpy="0 0.0 3.14"/>
     <parent link="base_link"/>
     <child link="laser_link"/>
     <axis xyz="0.0 0.0 1.0"/>
   </joint>
-    <!-- 2D LIDAR-->
+    <!-- 2D LIDAR
   <gazebo reference="laser_link">
     <sensor name="lidar" type="gpu_lidar">
@@ -219,6 +272,5 @@
       </lidar>
     </sensor>
-  </gazebo>
-<!--
+  </gazebo>-->
   <gazebo reference="laser_link">
     <sensor type="gpu_lidar" name="generic_lidar_sensor">
@@ -280,5 +332,4 @@
     </sensor>
   </gazebo>
--->
   <joint name="navsat_joint" type="fixed">
     <origin xyz="0 0 0" rpy="0 0 0" />
