Commit message: updates
new urdf + world

File: bot_description/urdf/bot.urdf.xacro (robot description, xacro)
@@ -1,4 +1,4 @@
 <?xml version="1.0" ?>
-  <robot name="bot" xmlns:xacro="http://ros.org/wiki/xacro">
+<robot name="bot" xmlns:xacro="http://ros.org/wiki/xacro">
   <xacro:include filename="bot_ros2_control.xacro" />
   <link name="base_footprint">
@@ -7,106 +7,106 @@
     <parent link="base_footprint"/>
     <child link="base_link"/>
-    <origin xyz="0.0 0.0 0.15" rpy="0.0 0.0 3.14159"/>
-  </joint>
-<link name="base_link">
-  <visual>
-    <geometry>
-      <box size="0.8 0.7 0.2"/>
-    </geometry>
-    <material name="gray">
-      <color rgba="0.2 0.2 0.2 1" />
-    </material>
-  </visual>
-  <collision>
-    <geometry>
-      <box size="0.8 0.7 0.2"/>
-    </geometry>
-  </collision>
-  <inertial>
-    <mass value="2"/>
-    <inertia ixx="0.0817" iyy="0.1067" izz="0.18" ixy="0.0" ixz="0.0" iyz="0.0"/>
-  </inertial>
-</link>
+    <origin xyz="0.0 0.0 0.50" rpy="0.0 0.0 3.14159"/>
+  </joint>
+  <link name="base_link">
+    <visual>
+      <geometry>
+        <box size="1.6 1.2 0.35"/>
+      </geometry>
+      <material name="gray">
+        <color rgba="0.2 0.2 0.2 1" />
+      </material>
+    </visual>
+    <collision>
+      <geometry>
+        <box size="1.6 1.2 0.35"/>
+      </geometry>
+    </collision>
+    <inertial>
+      <mass value="80"/>
+      <inertia ixx="15.0" iyy="22.0" izz="35.0" ixy="0.0" ixz="0.0" iyz="0.0"/>
+    </inertial>
+  </link>
   <link name="wheel_front_right">
-  <inertial>
-    <mass value="0.5"/>  <!-- OK for small wheels -->
-    <inertia ixx="0.00156" iyy="0.00156" izz="0.0025" ixy="0.0" ixz="0.0" iyz="0.0"/>
-  </inertial>
-  <visual>
-    <geometry>
-      <cylinder radius="0.10" length="0.05"/>
-    </geometry>
-    <material name="white">
-      <color rgba="1 1 1 1"/>
-    </material>
-  </visual>
-  <collision>
-    <geometry>
-      <cylinder radius="0.10" length="0.05"/>
-    </geometry>
-  </collision>
+    <inertial>
+      <mass value="8.0"/>
+      <inertia ixx="0.18" iyy="0.18" izz="0.32" ixy="0.0" ixz="0.0" iyz="0.0"/>
+    </inertial>
+    <visual>
+      <geometry>
+        <cylinder radius="0.28" length="0.20"/>
+      </geometry>
+      <material name="black">
+        <color rgba="0.1 0.1 0.1 1"/>
+      </material>
+    </visual>
+    <collision>
+      <geometry>
+        <cylinder radius="0.28" length="0.20"/>
+      </geometry>
+    </collision>
   </link>
   <link name="wheel_front_left">
-  <inertial>
-    <mass value="0.5"/>
-    <inertia ixx="0.00156" iyy="0.00156" izz="0.0025" ixy="0.0" ixz="0.0" iyz="0.0"/>
-  </inertial>
-  <visual>
-    <geometry>
-      <cylinder radius="0.10" length="0.05"/>
-    </geometry>
-    <material name="white">
-      <color rgba="1 1 1 1"/>
-    </material>
-  </visual>
-  <collision>
-    <geometry>
-      <cylinder radius="0.10" length="0.05"/>
-    </geometry>
-  </collision>
-  </link>
-<link name="wheel_back_right">
-  <inertial>
-    <mass value="0.5"/>
-    <inertia ixx="0.00156" iyy="0.00156" izz="0.0025" ixy="0.0" ixz="0.0" iyz="0.0"/>
-  </inertial>
-  <visual>
-    <geometry>
-      <cylinder radius="0.10" length="0.05"/>
-    </geometry>
-    <material name="white">
-      <color rgba="1 1 1 1"/>
-    </material>
-  </visual>
-  <collision>
-    <geometry>
-      <cylinder radius="0.10" length="0.05"/>
-    </geometry>
-  </collision>
-  </link>
-<link name="wheel_back_left">
-  <inertial>
-    <mass value="0.5"/>
-    <inertia ixx="0.00156" iyy="0.00156" izz="0.0025" ixy="0.0" ixz="0.0" iyz="0.0"/>
-  </inertial>
-  <visual>
-    <geometry>
-      <cylinder radius="0.10" length="0.05"/>
-    </geometry>
-    <material name="white">
-      <color rgba="1 1 1 1"/>
-    </material>
-  </visual>
-  <collision>
-    <geometry>
-      <cylinder radius="0.10" length="0.05"/>
-    </geometry>
-  </collision>
-</link>
+    <inertial>
+      <mass value="8.0"/>
+      <inertia ixx="0.18" iyy="0.18" izz="0.32" ixy="0.0" ixz="0.0" iyz="0.0"/>
+    </inertial>
+    <visual>
+      <geometry>
+        <cylinder radius="0.28" length="0.20"/>
+      </geometry>
+      <material name="black">
+        <color rgba="0.1 0.1 0.1 1"/>
+      </material>
+    </visual>
+    <collision>
+      <geometry>
+        <cylinder radius="0.28" length="0.20"/>
+      </geometry>
+    </collision>
+  </link>
+  <link name="wheel_back_right">
+    <inertial>
+      <mass value="8.0"/>
+      <inertia ixx="0.18" iyy="0.18" izz="0.32" ixy="0.0" ixz="0.0" iyz="0.0"/>
+    </inertial>
+    <visual>
+      <geometry>
+        <cylinder radius="0.28" length="0.20"/>
+      </geometry>
+      <material name="black">
+        <color rgba="0.1 0.1 0.1 1"/>
+      </material>
+    </visual>
+    <collision>
+      <geometry>
+        <cylinder radius="0.28" length="0.20"/>
+      </geometry>
+    </collision>
+  </link>
+  <link name="wheel_back_left">
+    <inertial>
+      <mass value="8.0"/>
+      <inertia ixx="0.18" iyy="0.18" izz="0.32" ixy="0.0" ixz="0.0" iyz="0.0"/>
+    </inertial>
+    <visual>
+      <geometry>
+        <cylinder radius="0.28" length="0.20"/>
+      </geometry>
+      <material name="black">
+        <color rgba="0.1 0.1 0.1 1"/>
+      </material>
+    </visual>
+    <collision>
+      <geometry>
+        <cylinder radius="0.28" length="0.20"/>
+      </geometry>
+    </collision>
+  </link>
   <link name="rgb_camera">
     <inertial>
-            <mass value="0.05" />
-            <inertia ixx="0.01" ixy="0.0" ixz="0"
-            iyy="0.01" iyz="0" izz="0.01" />
+      <mass value="0.05" />
+      <inertia ixx="0.01" ixy="0.0" ixz="0"
+      iyy="0.01" iyz="0" izz="0.01" />
     </inertial>
     <visual>
@@ -117,13 +117,14 @@
         <color rgba="0 0 1 1"/>
       </material>
-    </visual>    <origin xyz="-0.35 0 0.15" rpy="0 0.0 3.14"/>
-    <collision>
-      <geometry>
-          <box size="0.1 0.1 0.1"/>
+    </visual>
+    <origin xyz="-0.35 0 0.15" rpy="0 0.0 3.14"/>
+    <collision>
+      <geometry>
+        <box size="0.1 0.1 0.1"/>
       </geometry>
     </collision>
   </link>
   <joint name="camera_joint" type="fixed">
-    <origin xyz="-0.43 0 0.0" rpy="0 0.0 3.14"/>
+    <origin xyz="-0.85 0 0.0" rpy="0 0.0 3.14"/>
     <parent link="base_link"/>
     <child link="rgb_camera"/>
@@ -137,5 +138,5 @@
   <link name="camera_link_optical">
   </link>
-    <gazebo reference="rgb_camera">
+  <gazebo reference="rgb_camera">
     <sensor name="camera" type="camera">
       <camera>
@@ -163,10 +164,10 @@
       <topic>camera/image_raw</topic>
     </sensor>
-    </gazebo>
+  </gazebo>
   <link name="thermal_camera">
     <inertial>
-            <mass value="0.05" />
-            <inertia ixx="0.01" ixy="0.0" ixz="0"
-            iyy="0.01" iyz="0" izz="0.01" />
+      <mass value="0.05" />
+      <inertia ixx="0.01" ixy="0.0" ixz="0"
+      iyy="0.01" iyz="0" izz="0.01" />
     </inertial>
     <visual>
@@ -177,13 +178,14 @@
         <color rgba="0 0 1 1"/>
       </material>
-    </visual>    <origin xyz="-0.35 0 0.15" rpy="0 0.0 3.14"/>
-    <collision>
-      <geometry>
-          <box size="0.1 0.1 0.1"/>
+    </visual>
+    <origin xyz="-0.35 0 0.15" rpy="0 0.0 3.14"/>
+    <collision>
+      <geometry>
+        <box size="0.1 0.1 0.1"/>
       </geometry>
     </collision>
   </link>
   <joint name="thermal_camera_joint" type="fixed">
-    <origin xyz="-0.43 0 0.15" rpy="0 0.0 3.14"/>
+    <origin xyz="-0.85 0 0.20" rpy="0 0.0 3.14"/>
     <parent link="base_link"/>
     <child link="thermal_camera"/>
@@ -217,89 +219,110 @@
     </sensor>
   </gazebo>
+  <link name="lidar_base">
+    <inertial>
+      <mass value="0.2" />
+      <inertia ixx="0.005" ixy="0.0" ixz="0"
+      iyy="0.005" iyz="0" izz="0.005" />
+    </inertial>
+    <visual>
+      <geometry>
+        <cylinder radius="0.08" length="0.06"/>
+      </geometry>
+      <material name="dark_gray">
+        <color rgba="0.3 0.3 0.3 1"/>
+      </material>
+    </visual>
+    <collision>
+      <geometry>
+        <cylinder radius="0.08" length="0.06"/>
+      </geometry>
+    </collision>
+  </link>
+  <joint name="lidar_base_joint" type="fixed">
+    <origin xyz="0 0 0.52" rpy="0 0.0 0"/>
+    <parent link="base_link"/>
+    <child link="lidar_base"/>
+  </joint>
   <link name="laser_link">
     <inertial>
-            <mass value="0.5" />
-            <inertia ixx="0.01" ixy="0.0" ixz="0"
-            iyy="0.01" iyz="0" izz="0.01" />
-    </inertial>
-    <visual>
-      <geometry>
-        <cylinder radius="0.1" length="0.1"/>
-      </geometry>
-      <material name="red">
-        <color rgba="1 0 0  1"/>
-      </material>
-    </visual>
-    <collision>
-      <geometry>
-        <cylinder radius="0.1" length="0.1"/>
-      </geometry>
-    </collision>
-  </link>
-  <joint name="laser_joint" type="fixed">
-    <origin xyz="0 0 0.3" rpy="0 0.0 3.14"/>
-    <parent link="base_link"/>
+      <mass value="0.3" />
+      <inertia ixx="0.008" ixy="0.0" ixz="0"
+      iyy="0.008" iyz="0" izz="0.012" />
+    </inertial>
+    <visual>
+      <geometry>
+        <cylinder radius="0.06" length="0.08"/>
+      </geometry>
+      <material name="lidar_black">
+        <color rgba="0.1 0.1 0.1 1"/>
+      </material>
+    </visual>
+    <collision>
+      <geometry>
+        <cylinder radius="0.06" length="0.08"/>
+      </geometry>
+    </collision>
+  </link>
+  <link name="lidar_dome">
+    <inertial>
+      <mass value="0.1" />
+      <inertia ixx="0.002" ixy="0.0" ixz="0"
+      iyy="0.002" iyz="0" izz="0.002" />
+    </inertial>
+    <visual>
+      <geometry>
+        <sphere radius="0.055"/>
+      </geometry>
+      <material name="lidar_transparent">
+        <color rgba="0.2 0.2 0.2 0.6"/>
+      </material>
+    </visual>
+    <collision>
+      <geometry>
+        <sphere radius="0.055"/>
+      </geometry>
+    </collision>
+  </link>
+  <joint name="laser_joint" type="continuous">
+    <origin xyz="0 0 0.03" rpy="0 0.0 0"/>
+    <parent link="lidar_base"/>
     <child link="laser_link"/>
     <axis xyz="0.0 0.0 1.0"/>
-  </joint>
-    <!-- 2D LIDAR
+    <dynamics damping="0.1" friction="0.1"/>
+  </joint>
+  <joint name="lidar_dome_joint" type="fixed">
+    <origin xyz="0 0 0.04" rpy="0 0.0 0"/>
+    <parent link="laser_link"/>
+    <child link="lidar_dome"/>
+  </joint>
   <gazebo reference="laser_link">
-    <sensor name="lidar" type="gpu_lidar">
+    <sensor type="gpu_lidar" name="generic_lidar_sensor">
+      <update_rate>50</update_rate>
+      <visualize>true</visualize>
       <always_on>true</always_on>
-      <visualize>true</visualize>
-      <topic>scan</topic>
-      <update_rate>5</update_rate>
-      <gz_frame_id>laser_link</gz_frame_id>
+      <frame_id>laser_link</frame_id>
+      <ignition_frame_id>laser_link</ignition_frame_id>
+      <topic>/scan/points</topic>
       <lidar>
         <scan>
           <horizontal>
-            <samples>360</samples>
-            <resolution>1.00000</resolution>
-            <min_angle>0.000000</min_angle>
-            <max_angle>6.280000</max_angle>
+            <samples>1800</samples>
+            <resolution>0.2</resolution>
+            <min_angle>-3.1415926</min_angle>
+            <max_angle>3.1415926</max_angle>
           </horizontal>
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
Commit message: new world

File: bot_description/urdf/bot.urdf.xacro (robot description, xacro)
@@ -219,29 +219,4 @@
     </sensor>
   </gazebo>
-  <link name="lidar_base">
-    <inertial>
-      <mass value="0.2" />
-      <inertia ixx="0.005" ixy="0.0" ixz="0"
-      iyy="0.005" iyz="0" izz="0.005" />
-    </inertial>
-    <visual>
-      <geometry>
-        <cylinder radius="0.08" length="0.06"/>
-      </geometry>
-      <material name="dark_gray">
-        <color rgba="0.3 0.3 0.3 1"/>
-      </material>
-    </visual>
-    <collision>
-      <geometry>
-        <cylinder radius="0.08" length="0.06"/>
-      </geometry>
-    </collision>
-  </link>
-  <joint name="lidar_base_joint" type="fixed">
-    <origin xyz="0 0 0.52" rpy="0 0.0 0"/>
-    <parent link="base_link"/>
-    <child link="lidar_base"/>
-  </joint>
   <link name="laser_link">
     <inertial>
@@ -264,35 +239,10 @@
     </collision>
   </link>
-  <link name="lidar_dome">
-    <inertial>
-      <mass value="0.1" />
-      <inertia ixx="0.002" ixy="0.0" ixz="0"
-      iyy="0.002" iyz="0" izz="0.002" />
-    </inertial>
-    <visual>
-      <geometry>
-        <sphere radius="0.055"/>
-      </geometry>
-      <material name="lidar_transparent">
-        <color rgba="0.2 0.2 0.2 0.6"/>
-      </material>
-    </visual>
-    <collision>
-      <geometry>
-        <sphere radius="0.055"/>
-      </geometry>
-    </collision>
-  </link>
   <joint name="laser_joint" type="continuous">
-    <origin xyz="0 0 0.03" rpy="0 0.0 0"/>
-    <parent link="lidar_base"/>
+    <origin xyz="0 0 0.3" rpy="0 0.0 0"/>
+    <parent link="base_link"/>
     <child link="laser_link"/>
     <axis xyz="0.0 0.0 1.0"/>
     <dynamics damping="0.1" friction="0.1"/>
-  </joint>
-  <joint name="lidar_dome_joint" type="fixed">
-    <origin xyz="0 0 0.04" rpy="0 0.0 0"/>
-    <parent link="laser_link"/>
-    <child link="lidar_dome"/>
   </joint>
   <gazebo reference="laser_link">
@@ -371,4 +321,6 @@
   <link name="navsat_link">
   </link>
+  <link name="imu_link">
+  </link>
   <joint name="imu_joint" type="fixed">
     <origin xyz="0 0 0" rpy="0 0 0" />
@@ -376,6 +328,4 @@
     <child link="imu_link" />
   </joint>
-  <link name="imu_link">
-  </link>
   <gazebo reference="imu_link">
     <sensor name="imu_sensor" type="imu">

Commit message: return node lifecycle

File: bot_description/urdf/bot.urdf.xacro (robot description, xacro)
@@ -314,4 +314,6 @@
     <material>Gazebo/GreyTransparent</material>
   </gazebo>
+  <link name="navsat_link">
+  </link>
   <joint name="navsat_joint" type="fixed">
     <origin xyz="0 0 0" rpy="0 0 0" />
@@ -319,6 +321,4 @@
     <child link="navsat_link" />
   </joint>
-  <link name="navsat_link">
-  </link>
   <link name="imu_link">
   </link>

Commit message: add pcd2pgm pkg

File: bot_description/urdf/bot.urdf.xacro (robot description, xacro)
@@ -219,5 +219,5 @@
     </sensor>
   </gazebo>
-  <link name="laser_link">
+  <link name="lidar_link">
     <inertial>
       <mass value="0.3" />
@@ -239,18 +239,18 @@
     </collision>
   </link>
-  <joint name="laser_joint" type="continuous">
+  <joint name="lidar_joint" type="continuous">
     <origin xyz="0 0 0.3" rpy="0 0.0 0"/>
     <parent link="base_link"/>
-    <child link="laser_link"/>
+    <child link="lidar_link"/>
     <axis xyz="0.0 0.0 1.0"/>
     <dynamics damping="0.1" friction="0.1"/>
   </joint>
-  <gazebo reference="laser_link">
+  <gazebo reference="lidar_link">
     <sensor type="gpu_lidar" name="generic_lidar_sensor">
       <update_rate>50</update_rate>
       <visualize>true</visualize>
       <always_on>true</always_on>
-      <frame_id>laser_link</frame_id>
-      <ignition_frame_id>laser_link</ignition_frame_id>
+      <frame_id>lidar_link</frame_id>
+      <ignition_frame_id>lidar_link</ignition_frame_id>
       <topic>/scan/points</topic>
       <lidar>
@@ -278,6 +278,6 @@
     <sensor type="gpu_lidar" name="generic_twold_lidar_sensor">
       <topic>/scan</topic>
-      <frame_id>laser_link</frame_id>
-      <ignition_frame_id>laser_link</ignition_frame_id>
+      <frame_id>lidar_link</frame_id>
+      <ignition_frame_id>lidar_link</ignition_frame_id>
       <update_rate>50.0</update_rate>
       <ray>
@@ -305,12 +305,6 @@
     </sensor>
   </gazebo>
-  <gazebo reference="lidar_base">
-    <material>Gazebo/DarkGrey</material>
-  </gazebo>
-  <gazebo reference="laser_link">
+  <gazebo reference="lidar_link">
     <material>Gazebo/Black</material>
-  </gazebo>
-  <gazebo reference="lidar_dome">
-    <material>Gazebo/GreyTransparent</material>
   </gazebo>
   <link name="navsat_link">

Commit message: fixes

File: bot_description/urdf/bot.urdf.xacro (robot description, xacro)
@@ -219,5 +219,5 @@
     </sensor>
   </gazebo>
-  <link name="lidar_link">
+  <link name="laser_link">
     <inertial>
       <mass value="0.3" />
@@ -239,18 +239,18 @@
     </collision>
   </link>
-  <joint name="lidar_joint" type="continuous">
+  <joint name="laser_joint" type="continuous">
     <origin xyz="0 0 0.3" rpy="0 0.0 0"/>
     <parent link="base_link"/>
-    <child link="lidar_link"/>
+    <child link="laser_link"/>
     <axis xyz="0.0 0.0 1.0"/>
     <dynamics damping="0.1" friction="0.1"/>
   </joint>
-  <gazebo reference="lidar_link">
+  <gazebo reference="laser_link">
     <sensor type="gpu_lidar" name="generic_lidar_sensor">
       <update_rate>50</update_rate>
       <visualize>true</visualize>
       <always_on>true</always_on>
-      <frame_id>lidar_link</frame_id>
-      <ignition_frame_id>lidar_link</ignition_frame_id>
+      <frame_id>laser_link</frame_id>
+      <ignition_frame_id>laser_link</ignition_frame_id>
       <topic>/scan/points</topic>
       <lidar>
@@ -278,6 +278,6 @@
     <sensor type="gpu_lidar" name="generic_twold_lidar_sensor">
       <topic>/scan</topic>
-      <frame_id>lidar_link</frame_id>
-      <ignition_frame_id>lidar_link</ignition_frame_id>
+      <frame_id>laser_link</frame_id>
+      <ignition_frame_id>laser_link</ignition_frame_id>
       <update_rate>50.0</update_rate>
       <ray>
@@ -305,6 +305,12 @@
     </sensor>
   </gazebo>
-  <gazebo reference="lidar_link">
+  <gazebo reference="lidar_base">
+    <material>Gazebo/DarkGrey</material>
+  </gazebo>
+  <gazebo reference="laser_link">
     <material>Gazebo/Black</material>
+  </gazebo>
+  <gazebo reference="lidar_dome">
+    <material>Gazebo/GreyTransparent</material>
   </gazebo>
   <link name="navsat_link">
