Commit message: confidence engine

File: bot_description/urdf/bot.urdf.xacro (robot description, xacro)
@@ -1,4 +1,4 @@
 <?xml version="1.0" ?>
-<robot name="bot" xmlns:xacro="http://ros.org/wiki/xacro">
+  <robot name="bot" xmlns:xacro="http://ros.org/wiki/xacro">
   <xacro:include filename="bot_ros2_control.xacro" />
   <link name="base_footprint">
@@ -7,106 +7,106 @@
     <parent link="base_footprint"/>
     <child link="base_link"/>
-    <origin xyz="0.0 0.0 0.50" rpy="0.0 0.0 3.14159"/>
-  </joint>
-  <link name="base_link">
-    <visual>
-      <geometry>
-        <box size="1.6 1.2 0.35"/>
-      </geometry>
-      <material name="gray">
-        <color rgba="0.2 0.2 0.2 1" />
-      </material>
-    </visual>
-    <collision>
-      <geometry>
-        <box size="1.6 1.2 0.35"/>
-      </geometry>
-    </collision>
-    <inertial>
-      <mass value="80"/>
-      <inertia ixx="15.0" iyy="22.0" izz="35.0" ixy="0.0" ixz="0.0" iyz="0.0"/>
-    </inertial>
-  </link>
+    <origin xyz="0.0 0.0 0.15" rpy="0.0 0.0 3.14159"/>
+  </joint>
+<link name="base_link">
+  <visual>
+    <geometry>
+      <box size="0.8 0.7 0.2"/>
+    </geometry>
+    <material name="gray">
+      <color rgba="0.2 0.2 0.2 1" />
+    </material>
+  </visual>
+  <collision>
+    <geometry>
+      <box size="0.8 0.7 0.2"/>
+    </geometry>
+  </collision>
+  <inertial>
+    <mass value="2"/>
+    <inertia ixx="0.0817" iyy="0.1067" izz="0.18" ixy="0.0" ixz="0.0" iyz="0.0"/>
+  </inertial>
+</link>
   <link name="wheel_front_right">
-    <inertial>
-      <mass value="8.0"/>
-      <inertia ixx="0.18" iyy="0.18" izz="0.32" ixy="0.0" ixz="0.0" iyz="0.0"/>
-    </inertial>
-    <visual>
-      <geometry>
-        <cylinder radius="0.28" length="0.20"/>
-      </geometry>
-      <material name="black">
-        <color rgba="0.1 0.1 0.1 1"/>
-      </material>
-    </visual>
-    <collision>
-      <geometry>
-        <cylinder radius="0.28" length="0.20"/>
-      </geometry>
-    </collision>
+  <inertial>
+    <mass value="0.5"/>  <!-- OK for small wheels -->
+    <inertia ixx="0.00156" iyy="0.00156" izz="0.0025" ixy="0.0" ixz="0.0" iyz="0.0"/>
+  </inertial>
+  <visual>
+    <geometry>
+      <cylinder radius="0.10" length="0.05"/>
+    </geometry>
+    <material name="white">
+      <color rgba="1 1 1 1"/>
+    </material>
+  </visual>
+  <collision>
+    <geometry>
+      <cylinder radius="0.10" length="0.05"/>
+    </geometry>
+  </collision>
   </link>
   <link name="wheel_front_left">
-    <inertial>
-      <mass value="8.0"/>
-      <inertia ixx="0.18" iyy="0.18" izz="0.32" ixy="0.0" ixz="0.0" iyz="0.0"/>
-    </inertial>
-    <visual>
-      <geometry>
-        <cylinder radius="0.28" length="0.20"/>
-      </geometry>
-      <material name="black">
-        <color rgba="0.1 0.1 0.1 1"/>
-      </material>
-    </visual>
-    <collision>
-      <geometry>
-        <cylinder radius="0.28" length="0.20"/>
-      </geometry>
-    </collision>
-  </link>
-  <link name="wheel_back_right">
-    <inertial>
-      <mass value="8.0"/>
-      <inertia ixx="0.18" iyy="0.18" izz="0.32" ixy="0.0" ixz="0.0" iyz="0.0"/>
-    </inertial>
-    <visual>
-      <geometry>
-        <cylinder radius="0.28" length="0.20"/>
-      </geometry>
-      <material name="black">
-        <color rgba="0.1 0.1 0.1 1"/>
-      </material>
-    </visual>
-    <collision>
-      <geometry>
-        <cylinder radius="0.28" length="0.20"/>
-      </geometry>
-    </collision>
-  </link>
-  <link name="wheel_back_left">
-    <inertial>
-      <mass value="8.0"/>
-      <inertia ixx="0.18" iyy="0.18" izz="0.32" ixy="0.0" ixz="0.0" iyz="0.0"/>
-    </inertial>
-    <visual>
-      <geometry>
-        <cylinder radius="0.28" length="0.20"/>
-      </geometry>
-      <material name="black">
-        <color rgba="0.1 0.1 0.1 1"/>
-      </material>
-    </visual>
-    <collision>
-      <geometry>
-        <cylinder radius="0.28" length="0.20"/>
-      </geometry>
-    </collision>
-  </link>
+  <inertial>
+    <mass value="0.5"/>
+    <inertia ixx="0.00156" iyy="0.00156" izz="0.0025" ixy="0.0" ixz="0.0" iyz="0.0"/>
+  </inertial>
+  <visual>
+    <geometry>
+      <cylinder radius="0.10" length="0.05"/>
+    </geometry>
+    <material name="white">
+      <color rgba="1 1 1 1"/>
+    </material>
+  </visual>
+  <collision>
+    <geometry>
+      <cylinder radius="0.10" length="0.05"/>
+    </geometry>
+  </collision>
+  </link>
+<link name="wheel_back_right">
+  <inertial>
+    <mass value="0.5"/>
+    <inertia ixx="0.00156" iyy="0.00156" izz="0.0025" ixy="0.0" ixz="0.0" iyz="0.0"/>
+  </inertial>
+  <visual>
+    <geometry>
+      <cylinder radius="0.10" length="0.05"/>
+    </geometry>
+    <material name="white">
+      <color rgba="1 1 1 1"/>
+    </material>
+  </visual>
+  <collision>
+    <geometry>
+      <cylinder radius="0.10" length="0.05"/>
+    </geometry>
+  </collision>
+  </link>
+<link name="wheel_back_left">
+  <inertial>
+    <mass value="0.5"/>
+    <inertia ixx="0.00156" iyy="0.00156" izz="0.0025" ixy="0.0" ixz="0.0" iyz="0.0"/>
+  </inertial>
+  <visual>
+    <geometry>
+      <cylinder radius="0.10" length="0.05"/>
+    </geometry>
+    <material name="white">
+      <color rgba="1 1 1 1"/>
+    </material>
+  </visual>
+  <collision>
+    <geometry>
+      <cylinder radius="0.10" length="0.05"/>
+    </geometry>
+  </collision>
+</link>
   <link name="rgb_camera">
     <inertial>
-      <mass value="0.05" />
-      <inertia ixx="0.01" ixy="0.0" ixz="0"
-      iyy="0.01" iyz="0" izz="0.01" />
+            <mass value="0.05" />
+            <inertia ixx="0.01" ixy="0.0" ixz="0"
+            iyy="0.01" iyz="0" izz="0.01" />
     </inertial>
     <visual>
@@ -117,14 +117,13 @@
         <color rgba="0 0 1 1"/>
       </material>
-    </visual>
-    <origin xyz="-0.35 0 0.15" rpy="0 0.0 3.14"/>
+    </visual>    <origin xyz="-0.35 0 0.15" rpy="0 0.0 3.14"/>
     <collision>
       <geometry>
-        <box size="0.1 0.1 0.1"/>
+          <box size="0.1 0.1 0.1"/>
       </geometry>
     </collision>
   </link>
   <joint name="camera_joint" type="fixed">
-    <origin xyz="-0.85 0 0.0" rpy="0 0.0 3.14"/>
+    <origin xyz="-0.43 0 0.0" rpy="0 0.0 3.14"/>
     <parent link="base_link"/>
     <child link="rgb_camera"/>
@@ -138,5 +137,5 @@
   <link name="camera_link_optical">
   </link>
-  <gazebo reference="rgb_camera">
+    <gazebo reference="rgb_camera">
     <sensor name="camera" type="camera">
       <camera>
@@ -164,10 +163,10 @@
       <topic>camera/image_raw</topic>
     </sensor>
-  </gazebo>
+    </gazebo>
   <link name="thermal_camera">
     <inertial>
-      <mass value="0.05" />
-      <inertia ixx="0.01" ixy="0.0" ixz="0"
-      iyy="0.01" iyz="0" izz="0.01" />
+            <mass value="0.05" />
+            <inertia ixx="0.01" ixy="0.0" ixz="0"
+            iyy="0.01" iyz="0" izz="0.01" />
     </inertial>
     <visual>
@@ -178,14 +177,13 @@
         <color rgba="0 0 1 1"/>
       </material>
-    </visual>
-    <origin xyz="-0.35 0 0.15" rpy="0 0.0 3.14"/>
+    </visual>    <origin xyz="-0.35 0 0.15" rpy="0 0.0 3.14"/>
     <collision>
       <geometry>
-        <box size="0.1 0.1 0.1"/>
+          <box size="0.1 0.1 0.1"/>
       </geometry>
     </collision>
   </link>
   <joint name="thermal_camera_joint" type="fixed">
-    <origin xyz="-0.85 0 0.20" rpy="0 0.0 3.14"/>
+    <origin xyz="-0.43 0 0.15" rpy="0 0.0 3.14"/>
     <parent link="base_link"/>
     <child link="thermal_camera"/>
@@ -221,58 +219,87 @@
   <link name="laser_link">
     <inertial>
-      <mass value="0.3" />
-      <inertia ixx="0.008" ixy="0.0" ixz="0"
-      iyy="0.008" iyz="0" izz="0.012" />
+            <mass value="0.5" />
+            <inertia ixx="0.01" ixy="0.0" ixz="0"
+            iyy="0.01" iyz="0" izz="0.01" />
     </inertial>
     <visual>
       <geometry>
-        <cylinder radius="0.06" length="0.08"/>
-      </geometry>
-      <material name="lidar_black">
-        <color rgba="0.1 0.1 0.1 1"/>
+        <cylinder radius="0.1" length="0.1"/>
+      </geometry>
+      <material name="red">
+        <color rgba="1 0 0  1"/>
       </material>
     </visual>
     <collision>
       <geometry>
-        <cylinder radius="0.06" length="0.08"/>
+        <cylinder radius="0.1" length="0.1"/>
       </geometry>
     </collision>
   </link>
-  <joint name="laser_joint" type="continuous">
-    <origin xyz="0 0 0.3" rpy="0 0.0 0"/>
+  <joint name="laser_joint" type="fixed">
+    <origin xyz="0 0 0.3" rpy="0 0.0 3.14"/>
     <parent link="base_link"/>
     <child link="laser_link"/>
     <axis xyz="0.0 0.0 1.0"/>
-    <dynamics damping="0.1" friction="0.1"/>
-  </joint>
+  </joint>
+    <!-- 2D LIDAR
   <gazebo reference="laser_link">
-    <sensor type="gpu_lidar" name="generic_lidar_sensor">
-      <update_rate>50</update_rate>
+    <sensor name="lidar" type="gpu_lidar">
+      <always_on>true</always_on>
       <visualize>true</visualize>
-      <always_on>true</always_on>
-      <frame_id>laser_link</frame_id>
-      <ignition_frame_id>laser_link</ignition_frame_id>
-      <topic>/scan/points</topic>
+      <topic>scan</topic>
+      <update_rate>5</update_rate>
+      <gz_frame_id>laser_link</gz_frame_id>
       <lidar>
         <scan>
           <horizontal>
-            <samples>1800</samples>
-            <resolution>0.2</resolution>
-            <min_angle>-3.1415926</min_angle>
-            <max_angle>3.1415926</max_angle>
+            <samples>360</samples>
+            <resolution>1.00000</resolution>
+            <min_angle>0.000000</min_angle>
+            <max_angle>6.280000</max_angle>
           </horizontal>
-          <vertical>
-            <samples>16</samples>
-            <resolution>2</resolution>
-            <min_angle>-0.261799</min_angle>
-            <max_angle>0.261799</max_angle>
-          </vertical>
         </scan>
         <range>
-          <min>0.3</min>
-          <max>100</max>
-          <resolution>0.001</resolution>
+          <min>0.120000</min>
+          <max>12.0</max>
+          <resolution>0.02</resolution>
         </range>
+        <noise>
+          <type>gaussian</type>
+          <mean>0.0</mean>
+          <stddev>0.01</stddev>
+        </noise>
       </lidar>
+    </sensor>
+  </gazebo>-->
+  <gazebo reference="laser_link">
+    <sensor type="gpu_lidar" name="generic_lidar_sensor">
+        <update_rate>50</update_rate>
+        <visualize>true</visualize>
+        <always_on>true</always_on>
+        <frame_id>laser_link</frame_id>
+        <ignition_frame_id>laser_link</ignition_frame_id>
+        <topic>/scan/points</topic>
+        <lidar>
+          <scan>
+              <horizontal>
+                <samples>1800</samples>
+                <resolution>0.2</resolution>
+                <min_angle>-3.1415926</min_angle>
+                <max_angle>3.1415926</max_angle>
+              </horizontal>
+              <vertical>
+                <samples>16</samples>
+                <resolution>2</resolution>
+                <min_angle>-0.261799</min_angle>
+                <max_angle>0.261799</max_angle>
+              </vertical>
+            </scan>
+            <range>
+              <min>0.3</min>
+              <max>100</max>
+              <resolution>0.001</resolution>
+            </range>
+        </lidar>
     </sensor>
     <sensor type="gpu_lidar" name="generic_twold_lidar_sensor">
@@ -305,15 +332,4 @@
     </sensor>
   </gazebo>
-  <gazebo reference="lidar_base">
-    <material>Gazebo/DarkGrey</material>
-  </gazebo>
-  <gazebo reference="laser_link">
-    <material>Gazebo/Black</material>
-  </gazebo>
-  <gazebo reference="lidar_dome">
-    <material>Gazebo/GreyTransparent</material>
-  </gazebo>
-  <link name="navsat_link">
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
Commit message: rule engine basic structure

File: bot_description/urdf/bot.urdf.xacro (robot description, xacro)
@@ -164,57 +164,4 @@
     </sensor>
     </gazebo>
-  <link name="thermal_camera">
-    <inertial>
-            <mass value="0.05" />
-            <inertia ixx="0.01" ixy="0.0" ixz="0"
-            iyy="0.01" iyz="0" izz="0.01" />
-    </inertial>
-    <visual>
-      <geometry>
-        <box size="0.1 0.1 0.1"/>
-      </geometry>
-      <material name="blue">
-        <color rgba="0 0 1 1"/>
-      </material>
-    </visual>    <origin xyz="-0.35 0 0.15" rpy="0 0.0 3.14"/>
-    <collision>
-      <geometry>
-          <box size="0.1 0.1 0.1"/>
-      </geometry>
-    </collision>
-  </link>
-  <joint name="thermal_camera_joint" type="fixed">
-    <origin xyz="-0.43 0 0.15" rpy="0 0.0 3.14"/>
-    <parent link="base_link"/>
-    <child link="thermal_camera"/>
-    <axis xyz="0.0 0 0"/>
-  </joint>
-  <gazebo reference="thermal_camera">
-    <sensor name="thermal_camera_8bit" type="thermal">
-      <camera>
-        <horizontal_fov>1.047</horizontal_fov>
-        <image>
-          <width>320</width>
-          <height>240</height>
-          <format>L8</format>
-        </image>
-        <clip>
-          <near>0.1</near>
-          <far>100</far>
-        </clip>
-      </camera>
-      <always_on>1</always_on>
-      <update_rate>30</update_rate>
-      <visualize>true</visualize>
-      <topic>thermal_camera_8bit/image</topic>
-      <plugin
-        filename="ignition-gazebo-thermal-sensor-system"
-        name="gz::sim::systems::ThermalSensor">
-        <min_temp>253.15</min_temp>
-        <max_temp>673.15</max_temp>
-        <resolution>3.0</resolution>
-      </plugin>
-    </sensor>
-  </gazebo>
   <link name="laser_link">
     <inertial>
