Commit message: Integrate lidarslam and traversability

File: LIO-SAM/config/robot.urdf.xacro (robot description, xacro)
@@ -2,32 +2,20 @@
 <robot name="lio" xmlns:xacro="http://tixiaoshan.github.io/">
   <xacro:property name="PI" value="3.1415926535897931" />
-  <link name="chassis_link"></link>
   <link name="base_link"></link>
-  <joint name="base_link_joint" type="fixed">
-    <parent link="base_link"/>
-    <child link="chassis_link" />
-    <origin xyz="0 0 0" rpy="0 0 0" />
-  </joint>
-  <link name="lidar_link"> </link>
-  <joint name="lidar_joint" type="fixed">
+  <link name="laser_link"> </link>
+  <joint name="laser_joint" type="fixed">
     <parent link="base_link" />
-    <child link="lidar_link" />
-    <origin xyz="0 0 0" rpy="0 0 0" />
+    <child link="laser_link" />
+    <origin xyz="0 0 0.45" rpy="0 0 0" />
   </joint>
   <link name="imu_link"> </link>
   <joint name="imu_joint" type="fixed">
-    <parent link="chassis_link" />
+    <parent link="base_link" />
     <child link="imu_link" />
-    <origin xyz="0 0 0" rpy="0 0 0" />
-  </joint>
-  <link name="laser_sensor_frame"> </link>
-  <joint name="laser_joint" type="fixed">
-    <parent link="imu_link" />
-    <child link="laser_sensor_frame" />
     <origin xyz="0 0 0" rpy="0 0 0" />
   </joint>
   <link name="navsat_link"> </link>
   <joint name="navsat_joint" type="fixed">
-    <parent link="chassis_link" />
+    <parent link="base_link" />
     <child link="navsat_link" />
     <origin xyz="0 0 0" rpy="0 0 0" />

File: bot_description/urdf/bot.urdf.xacro (robot description, xacro)
@@ -1,4 +1,5 @@
 <?xml version="1.0" ?>
 <robot name="bot" xmlns:xacro="http://ros.org/wiki/xacro">
+  <xacro:arg name="controller_params_file" default="$(find bot_controller)/config/bot_controller.yaml"/>
   <xacro:include filename="bot_ros2_control.xacro" />
   <xacro:property name="chassis_length" value="1.25"/>
@@ -15,5 +16,5 @@
   <xacro:property name="wheelbase" value="0.95"/>
   <xacro:property name="track_width" value="1.04"/>
-  <xacro:property name="lidar_mast_height" value="0.55"/>
+  <xacro:property name="lidar_mast_height" value="0.25"/>
   <xacro:property name="base_z" value="${ground_clearance + chassis_height / 2.0}"/>
   <xacro:property name="wheel_z" value="${wheel_radius - base_z}"/>
@@ -45,6 +46,6 @@
   <xacro:macro name="wheel_contact" params="link">
     <gazebo reference="${link}">
-      <mu1>1.4</mu1>
-      <mu2>0.9</mu2>
+      <mu1>1.2</mu1>
+      <mu2>0.8</mu2>
       <kp>500000.0</kp>
       <kd>50.0</kd>
@@ -54,11 +55,4 @@
     </gazebo>
   </xacro:macro>
-  <link name="base_footprint">
-  </link>
-  <joint name="base_joint" type="fixed">
-    <parent link="base_footprint"/>
-    <child link="base_link"/>
-    <origin xyz="0.0 0.0 ${base_z}" rpy="0.0 0.0 ${pi}"/>
-  </joint>
 <link name="base_link">
   <visual>
@@ -125,5 +119,5 @@
   </link>
   <joint name="camera_joint" type="fixed">
-    <origin xyz="${-chassis_length / 2.0 - 0.08} 0 ${chassis_height / 2.0 - 0.05}" rpy="0 0.0 ${pi}"/>
+    <origin xyz="${chassis_length / 2.0 + 0.08} 0 ${chassis_height / 2.0 - 0.05}" rpy="0 0 0"/>
     <parent link="base_link"/>
     <child link="rgbd_camera"/>
@@ -179,5 +173,5 @@
   </link>
   <joint name="laser_joint" type="fixed">
-    <origin xyz="0 0 ${chassis_height / 2.0 + lidar_mast_height}" rpy="0 0.0 ${pi}"/>
+    <origin xyz="0 0 ${chassis_height / 2.0 + lidar_mast_height}" rpy="0 0 0"/>
     <parent link="base_link"/>
     <child link="laser_link"/>
@@ -216,36 +210,36 @@
   <gazebo reference="laser_link">
     <sensor type="gpu_lidar" name="generic_lidar_sensor">
-        <update_rate>15</update_rate>
-        <visualize>false</visualize>
-        <always_on>true</always_on>
-        <frame_id>laser_link</frame_id>
-        <ignition_frame_id>laser_link</ignition_frame_id>
-        <topic>/lidar_3d</topic>
-        <lidar>
-          <scan>
-            <horizontal>
-              <samples>2400</samples>
-              <resolution>1.0</resolution>
-              <min_angle>-3.1415926</min_angle>
-              <max_angle>3.1415926</max_angle>
-            </horizontal>
-            <vertical>
-              <samples>32</samples>
-              <resolution>1.0</resolution>
-              <min_angle>-0.261799</min_angle>
-              <max_angle>0.261799</max_angle>
-            </vertical>
-          </scan>
-          <range>
-            <min>0.3</min>
-            <max>40</max>
-            <resolution>0.02</resolution>
-          </range>
-          <noise>
-            <type>gaussian</type>
-            <mean>0.0</mean>
-            <stddev>0.025</stddev>
-          </noise>
-        </lidar>
+      <update_rate>10</update_rate>
+      <visualize>true</visualize>
+      <always_on>true</always_on>
+      <frame_id>laser_link</frame_id>
+      <ignition_frame_id>laser_link</ignition_frame_id>
+      <topic>/lidar_3d</topic>
+      <lidar>
+        <scan>
+          <horizontal>
+            <samples>3600</samples>
+            <resolution>0.1</resolution>
+            <min_angle>-3.1415926</min_angle>
+            <max_angle>3.1415926</max_angle>
+          </horizontal>
+          <vertical>
+            <samples>32</samples>
+            <resolution>0.5</resolution>
+            <min_angle>-0.261799</min_angle>
+            <max_angle>0.261799</max_angle>
+          </vertical>
+        </scan>
+        <range>
+          <min>0.5</min>
+          <max>30.0</max>
+          <resolution>0.01</resolution>
+        </range>
+        <noise>
+          <type>gaussian</type>
+          <mean>0.0</mean>
+          <stddev>0.01</stddev>
+        </noise>
+      </lidar>
     </sensor>
     <sensor type="gpu_lidar" name="generic_twold_lidar_sensor">
@@ -365,26 +359,26 @@
   </gazebo>
   <joint name="wheel_front_right_joint" type="continuous">
+    <origin xyz="${wheelbase / 2.0} ${track_width / 2.0} ${wheel_z}" rpy="${pi / 2.0} 0.0 0.0"/>
+    <parent link="base_link"/>
+    <child link="wheel_front_right"/>
+    <axis xyz="0.0 0.0 -1.0"/>
+  </joint>
+  <joint name="wheel_front_left_joint" type="continuous">
+    <origin xyz="${wheelbase / 2.0} ${-track_width / 2.0} ${wheel_z}" rpy="${pi / 2.0} 0.0 0.0"/>
+    <parent link="base_link"/>
+    <child link="wheel_front_left"/>
+    <axis xyz="0.0 0.0 -1.0"/>
+  </joint>
+  <joint name="wheel_back_right_joint" type="continuous">
     <origin xyz="${-wheelbase / 2.0} ${track_width / 2.0} ${wheel_z}" rpy="${pi / 2.0} 0.0 0.0"/>
     <parent link="base_link"/>
-    <child link="wheel_front_right"/>
-    <axis xyz="0.0 0.0 1.0"/>
-  </joint>
-  <joint name="wheel_front_left_joint" type="continuous">
+    <child link="wheel_back_right"/>
+    <axis xyz="0.0 0.0 -1.0"/>
+  </joint>
+  <joint name="wheel_back_left_joint" type="continuous">
     <origin xyz="${-wheelbase / 2.0} ${-track_width / 2.0} ${wheel_z}" rpy="${pi / 2.0} 0.0 0.0"/>
     <parent link="base_link"/>
-    <child link="wheel_front_left"/>
-    <axis xyz="0.0 0.0 1.0"/>
-  </joint>
-  <joint name="wheel_back_right_joint" type="continuous">
-    <origin xyz="${wheelbase / 2.0} ${track_width / 2.0} ${wheel_z}" rpy="${pi / 2.0} 0.0 0.0"/>
-    <parent link="base_link"/>
-    <child link="wheel_back_right"/>
-    <axis xyz="0.0 0.0 1.0"/>
-  </joint>
-  <joint name="wheel_back_left_joint" type="continuous">
-    <origin xyz="${wheelbase / 2.0} ${-track_width / 2.0} ${wheel_z}" rpy="${pi / 2.0} 0.0 0.0"/>
-    <parent link="base_link"/>
     <child link="wheel_back_left"/>
-    <axis xyz="0.0 0.0 1.0"/>
+    <axis xyz="0.0 0.0 -1.0"/>
   </joint>
   <xacro:wheel_contact link="wheel_front_right"/>
@@ -394,5 +388,5 @@
     <gazebo>
         <plugin filename="ign_ros2_control-system" name="ign_ros2_control::IgnitionROS2ControlPlugin">
-            <parameters>$(find bot_controller)/config/bot_controller.yaml</parameters>
+            <parameters>$(arg controller_params_file)</parameters>
         </plugin>
         <plugin filename="libignition-gazebo-imu-system.so" name="ignition::gazebo::systems::Imu">
